File: Shift Register Sequencer.kicad_sch (KiCad schematic)
At the start: 111 parts, among them J1 Gate IN, J10 Step 4, J11 Step C, J12 Step 5, J13 Step F, J14 Step 0-F, J2 Step 0, J3 Step 6, J4 Step 1, J5 Step 7, J6 Step 2, J7 Step 8, J8 Step 3, J9 Step A, Q1 2N3904, Q2 2N3904, SW1 oneShot/continous, SW2 oneShot/continous, U1 4070, U2 SN74HC595N, U3 SN74HC595N, U4 TL072, U5 CD4050, U6 CD4050, U7 TL074, U8 4081, U9 TL074

Commit message: Minor fixes
Connections:
- net 0: no longer U6.3
- net 1: no longer U6.5
- net 2: no longer U6.7
- net 3: no longer U6.9
- net 4: no longer U6.11
- net 5: no longer U6.14
- net 6: now also U6.3
- net 7: now also U6.5
- net 8: now also U6.7
- net A: now also U6.9
- net C: now also U6.11
- net F: now also U6.14
Other:
- note added: "This mod sacrifices the gate option for a trigger on every clock cycle."
- note removed: "This mod sacrifices the gate option for a trigger on each clock."
Changed lines of the file:
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@@
   (text "*Use 1% resistors for Rf and Rg or \nhand pick similar values \nif exact output voltages are of a concern."
     (at 85.344 138.684 0)
-    (effects (font (size 0.6 0.6) italic) (justify left bottom))
+    (effects (font (size 0.7 0.7) italic) (justify left bottom))
   )
-  (text "This mod sacrifices the gate option \nfor a trigger on each clock."
+  (text "This mod sacrifices the gate option \nfor a trigger on every clock cycle."
     (at 32.512 129.286 0)
     (effects (font (size 1 1) italic) (justify left bottom))
@@
   )
   (text "*the current limiting resistors for the LEDs \ndepend on what kind of LEDs you use \nso I would experiment with those values before assembly."
-    (at 184.658 64.77 0)
-    (effects (font (size 0.6 0.6) italic) (justify left bottom))
+    (at 182.118 65.024 0)
+    (effects (font (size 0.7 0.7) italic) (justify left bottom))
   )
   (text "One Shot/Continous Select" (at 65.024 45.212 0)
@@
     )
   )
-  (global_label "2" (shape input) (at 352.552 68.326 180) (fields_autoplaced)
+  (global_label "8" (shape input) (at 352.552 68.326 180) (fields_autoplaced)
     (effects (font (size 1.27 1.27) (thickness 0.254) bold) (justify right))
     (property "Intersheet References" "${INTERSHEET_REFS}" (id 0) (at 348.8279 68.199 0)
@@
     )
   )
-  (global_label "4" (shape input) (at 352.552 85.598 180) (fields_autoplaced)
+  (global_label "C" (shape input) (at 352.552 85.598 180) (fields_autoplaced)
     (effects (font (size 1.27 1.27) (thickness 0.254) bold) (justify right))
-    (property "Intersheet References" "${INTERSHEET_REFS}" (id 0) (at 348.8279 85.471 0)
+    (property "Intersheet References" "${INTERSHEET_REFS}" (id 0) (at 348.7674 85.471 0)
       (effects (font (size 1.27 1.27) (thickness 0.254) bold) (justify right) hide)
     )
@@
     )
   )
-  (global_label "3" (shape input) (at 352.552 76.962 180) (fields_autoplaced)
+  (global_label "A" (shape input) (at 352.552 76.962 180) (fields_autoplaced)
     (effects (font (size 1.27 1.27) (thickness 0.254) bold) (justify right))
-    (property "Intersheet References" "${INTERSHEET_REFS}" (id 0) (at 348.8279 76.835 0)
+    (property "Intersheet References" "${INTERSHEET_REFS}" (id 0) (at 348.9488 76.835 0)
       (effects (font (size 1.27 1.27) (thickness 0.254) bold) (justify right) hide)
     )
@@
     )
   )
-  (global_label "0" (shape input) (at 352.552 51.054 180) (fields_autoplaced)
+  (global_label "6" (shape input) (at 352.552 51.054 180) (fields_autoplaced)
     (effects (font (size 1.27 1.27) (thickness 0.254) bold) (justify right))
     (property "Intersheet References" "${INTERSHEET_REFS}" (id 0) (at 348.8279 50.927 0)
@@
     )
   )
-  (global_label "1" (shape input) (at 352.552 59.69 180) (fields_autoplaced)
+  (global_label "7" (shape input) (at 352.552 59.69 180) (fields_autoplaced)
     (effects (font (size 1.27 1.27) (thickness 0.254) bold) (justify right))
     (property "Intersheet References" "${INTERSHEET_REFS}" (id 0) (at 348.8279 59.563 0)
@@
     )
   )
-  (global_label "5" (shape input) (at 352.552 94.234 180) (fields_autoplaced)
+  (global_label "F" (shape input) (at 352.552 94.234 180) (fields_autoplaced)
     (effects (font (size 1.27 1.27) (thickness 0.254) bold) (justify right))
-    (property "Intersheet References" "${INTERSHEET_REFS}" (id 0) (at 348.8279 94.107 0)
+    (property "Intersheet References" "${INTERSHEET_REFS}" (id 0) (at 348.9488 94.107 0)
       (effects (font (size 1.27 1.27) (thickness 0.254) bold) (justify right) hide)
     )
